File: Eagle/PCBs/Counter Toy/counter_toy.sch (EAGLE design)
At the start: 210 parts, among them Q1 2N7002, Q10 2N7002, Q100 2N7002, Q101 2N7002, Q102 2N7002, Q103 2N7002, Q104 2N7002, Q105 2N7002, Q106 2N7002, Q126 2N7002, Q127 2N7002, Q128 2N7002, Q129 2N7002, Q13 2N7002, Q130 2N7002, Q131 2N7002, Q132 2N7002, Q133 2N7002, Q134 2N7002, Q135 2N7002, Q136 2N7002, Q137 2N7002, Q138 2N7002, Q139 2N7002, Q14 2N7002, Q140 2N7002, Q141 2N7002, Q142 2N7002, Q15 2N7002, Q16 2N7002, Q162 2N7002, Q163 2N7002, Q164 2N7002, Q165 2N7002, Q166 2N7002, Q167 2N7002, Q168 2N7002, Q169 2N7002, Q17 2N7002, Q170 2N7002, Q171 2N7002, Q172 2N7002, Q173 2N7002, Q174 2N7002, Q175 2N7002, Q176 2N7002, Q177 2N7002, Q178 2N7002, Q198 2N7002, Q199 2N7002, Q200 2N7002, Q201 2N7002, Q202 2N7002, Q203 2N7002, Q204 2N7002, Q205 2N7002, Q206 2N7002, Q207 2N7002, Q208 2N7002, Q209 2N7002, Q21 2N7002, Q210 2N7002, Q211 2N7002, Q212 2N7002, Q213 2N7002, Q214 2N7002, Q22 2N7002, Q23 2N7002, Q234 2N7002, Q235 2N7002, Q236 2N7002, Q237 2N7002, Q238 2N7002, Q239 2N7002, Q240 2N7002, Q241 2N7002, Q242 2N7002, Q243 2N7002, Q244 2N7002, Q245 2N7002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

Commit message: Made DFF and byte more compact
Parts:
- removed D0, D1, D2, D3, D4, D5, D6, D7: TPPAD6, ellajameson-core:TPPAD6
- removed Q1, Q10, Q13, Q14, Q15, Q16, Q17, Q21, Q22, Q23, Q234, Q235, Q236, Q237, Q238, Q239, Q240, Q241, Q242, Q243, Q244, Q245, Q246, Q247, Q248, Q249, Q250, Q3, Q4, Q5, Q6, Q7, Q8, Q9: 2N7002, ellajameson-core:2N7002
- removed R104, R105, R106, R107, R108, R109, R110, R2, R3, R4, R5, R6, R7, R9: (no value), ellajameson-core:RES0603
- added I0, I1, I2, I3, I4, I5, I6, I7: TPPAD6, ellajameson-core:TPPAD6
- added Q11, Q12, Q18, Q19, Q2, Q20, Q24, Q25, Q26, Q27, Q28, Q29, Q30, Q31, Q32, Q33, Q34, Q72, Q73, Q74, Q75, Q76, Q77, Q78, Q79, Q80, Q81, Q82, Q83, Q84, Q85, Q86, Q87, Q88: 2N7002, ellajameson-core:2N7002
- added R1, R10, R11, R12, R13, R14, R32, R33, R34, R35, R36, R37, R38, R8: (no value), ellajameson-core:RES0603
Connections:
- removed net N$12: CLK.S, Q130.G, Q133.G, Q166.G, Q169.G, Q202.G, Q205.G, Q238.G, Q241.G, Q40.G, Q43.G, Q58.G, Q6.G, Q61.G, Q9.G, Q94.G, Q97.G
- removed net N$13: Q5.S, Q6.D
- removed net N$15: Q6.S, Q7.D
- removed net N$16: Q8.S, Q9.D
- removed net N$18: Q10.G, Q22.G, Q23.D, Q4.G, R9.1
- removed net N$2: Q1.G, Q21.G, Q5.D, R3.1
- removed net N$20: Q10.D, Q9.S
- removed net N$261: Q234.G, Q237.D, Q248.G, R105.1
- removed net N$262: Q234.D, Q239.G, Q243.G, R104.1
- removed net N$263: D7.S, Q235.G
- removed net N$264: Q234.S, Q235.D
- removed net N$265: Q235.S, Q236.D
- removed net N$266: Q237.G, Q240.D, Q244.G, Q245.G, R106.1
- removed net N$268: Q237.S, Q238.D
- removed net N$269: Q238.S, Q239.D
- removed net N$270: Q240.S, Q241.D
- removed net N$271: Q236.G, Q242.G, Q249.G, Q250.D, R110.1
- removed net N$272: Q241.S, Q242.D
- removed net N$273: Q240.G, Q243.D, R107.1
- removed net N$274: Q243.S, Q244.D
- removed net N$275: Q245.S, Q246.D
- removed net N$276: O7.S, Q245.D, Q247.G, R108.1
- removed net N$277: Q246.G, Q247.D, R109.1
- removed net N$278: Q247.S, Q248.D
- removed net N$279: Q248.S, Q249.D
- removed net N$28: Q13.D, Q8.G, R5.1
- removed net N$29: Q13.S, Q14.D
- removed net N$30: Q15.S, Q16.D
- removed net N$34: O0.S, Q15.D, Q17.G, R6.1
- removed net N$37: Q16.G, Q17.D, R7.1
- removed net N$38: Q17.S, Q21.D
- removed net N$39: Q21.S, Q22.D
- removed net N$40: Q106.G, Q142.G, Q178.G, Q214.G, Q23.G, Q250.G, Q52.G, Q70.G, R.S
- removed net N$5: Q1.D, Q13.G, Q7.G, R2.1
- removed net N$6: D0.S, Q3.G
- removed net N$7: Q1.S, Q3.D
- removed net N$8: Q3.S, Q4.D
- removed net N$9: Q14.G, Q15.G, Q5.G, Q8.D, R4.1
- new net N$1: Q18.D, Q2.G, Q32.G, R8.1
- new net N$10: Q11.D, Q2.S
- new net N$11: Q11.S, Q12.D
- new net N$14: Q18.G, Q24.D, Q28.G, Q29.G, R10.1
- new net N$17: CLK.S, Q130.G, Q133.G, Q166.G, Q169.G, Q19.G, Q202.G, Q205.G, Q25.G, Q40.G, Q43.G, Q58.G, Q61.G, Q76.G, Q79.G, Q94.G, Q97.G
- new net N$19: Q18.S, Q19.D
- new net N$21: Q19.S, Q20.D
- new net N$22: Q24.S, Q25.D
- new net N$23: Q12.G, Q26.G, Q33.G, Q34.D, R14.1
- new net N$24: Q25.S, Q26.D
- new net N$25: Q24.G, Q27.D, R11.1
- new net N$26: Q27.S, Q28.D
- new net N$27: Q29.S, Q30.D
- new net N$3: Q2.D, Q20.G, Q27.G, R1.1
- new net N$31: O7.S, Q29.D, Q31.G, R12.1
- new net N$32: Q30.G, Q31.D, R13.1
- new net N$33: Q31.S, Q32.D
- new net N$35: Q32.S, Q33.D
- new net N$36: Q106.G, Q142.G, Q178.G, Q214.G, Q34.G, Q52.G, Q70.G, Q88.G, R.S
- new net N$4: I7.S, Q11.G
- new net N$81: Q72.G, Q75.D, Q86.G, R33.1
- new net N$82: Q72.D, Q77.G, Q81.G, R32.1
- new net N$83: I3.S, Q73.G
- new net N$84: Q72.S, Q73.D
- new net N$85: Q73.S, Q74.D
- new net N$86: Q75.G, Q78.D, Q82.G, Q83.G, R34.1
- new net N$88: Q75.S, Q76.D
- new net N$89: Q76.S, Q77.D
- new net N$90: Q78.S, Q79.D
- new net N$91: Q74.G, Q80.G, Q87.G, Q88.D, R38.1
- new net N$92: Q79.S, Q80.D
- new net N$93: Q78.G, Q81.D, R35.1
- new net N$94: Q81.S, Q82.D
- new net N$95: Q83.S, Q84.D
- new net N$96: O3.S, Q83.D, Q85.G, R36.1
- new net N$97: Q84.G, Q85.D, R37.1
- new net N$98: Q85.S, Q86.D
- new net N$99: Q86.S, Q87.D
- net GND: now also Q12.S, Q20.S, Q26.S, Q28.S, Q30.S, Q33.S, Q34.S, Q74.S, Q77.S, Q80.S, Q82.S, Q84.S, Q87.S, Q88.S; no longer Q10.S, Q14.S, Q16.S, Q22.S, Q23.S, Q236.S, Q239.S, Q242.S, Q244.S, Q246.S, Q249.S, Q250.S, Q4.S, Q7.S
- net N$103: now also I4.S; no longer D3.S
- net N$116: now also O4.S; no longer O3.S
- net N$143: now also I2.S; no longer D4.S
- net N$156: now also O2.S; no longer O4.S
- net N$183: now also I1.S; no longer D5.S
- net N$196: now also O1.S; no longer O5.S
- net N$223: now also I0.S; no longer D6.S
- net N$236: now also O0.S; no longer O6.S
- net N$43: now also I5.S; no longer D2.S
- net N$56: now also O5.S; no longer O2.S
- net N$63: now also I6.S; no longer D1.S
- net N$76: now also O6.S; no longer O1.S
- net VCC: now also R1.2, R10.2, R11.2, R12.2, R13.2, R14.2, R32.2, R33.2, R34.2, R35.2, R36.2, R37.2, R38.2, R8.2; no longer R104.2, R105.2, R106.2, R107.2, R108.2, R109.2, R110.2, R2.2, R3.2, R4.2, R5.2, R6.2, R7.2, R9.2
Other:
- moved on the sheet: CLK, O0, O1, O2, O3, O4, O5, O6, O7, Q100, Q101, Q102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

Commit message: Made a button input and a multiplexer
Parts:
- removed CLK, I0, I1, I2, O0, O5, O6, O7, R: TPPAD6, ellajameson-core:TPPAD6
- removed Q100, Q101, Q102, Q103, Q104, Q105, Q106, Q12, Q126, Q127, Q128, Q129, Q130, Q131, Q132, Q133, Q134, Q135, Q136, Q137, Q138, Q139, Q140, Q141, Q142, Q162, Q163, Q164, Q165, Q166, Q167, Q168, Q169, Q170, Q171, Q172, Q173, Q174, Q175, Q176, Q177, Q178, Q198, Q199, Q200, Q201, Q202, Q203, Q204, Q205, Q206, Q207, Q208, Q209, Q210, Q211, Q212, Q213, Q214, Q31, Q32, Q33, Q34, Q36, Q37, Q38, Q39, Q40, Q41, Q42, Q43, Q44, Q45, Q46, Q47, Q48, Q49, Q50, Q51, Q52, Q54, Q55, Q56, Q57, Q58, Q59, Q60, Q61, Q62, Q63, Q64, Q65, Q66, Q67, Q68, Q69, Q70, Q72, Q73, Q74, Q75, Q76, Q77, Q78, Q79, Q80, Q81, Q82, Q83, Q84, Q85, Q86, Q87, Q88, Q90, Q91, Q92, Q93, Q94, Q95, Q96, Q97, Q98, Q99: 2N7002, ellajameson-core:2N7002
- removed R16, R17, R18, R19, R20, R21, R22, R24, R25, R26, R27, R28, R29, R30, R32, R33, R34, R35, R36, R37, R38, R40, R41, R42, R43, R44, R45, R46, R56, R57, R58, R59, R60, R61, R62, R72, R73, R74, R75, R76, R77, R78, R88, R89, R90, R91, R92, R93, R94: (no value), ellajameson-core:RES0603
- added I10, I8, I9, SEL1, SEL2, SEL3, SEL4: TPPAD6, ellajameson-core:TPPAD6
- added Q1, Q13, Q14, Q15, Q16, Q17, Q21, Q22, Q23, Q3, Q4, Q9: 2N7002, ellajameson-core:2N7002
- added R15, R3, R5, R7, R9: (no value), ellajameson-core:RES0603
Connections:
- removed net N$10: Q11.D, Q2.S
- removed net N$101: Q104.G, Q90.G, Q93.D, R41.1
- removed net N$102: Q90.D, Q95.G, Q99.G, R40.1
- removed net N$103: I4.S, Q91.G
- removed net N$104: Q90.S, Q91.D
- removed net N$105: Q91.S, Q92.D
- removed net N$106: Q100.G, Q101.G, Q93.G, Q96.D, R42.1
- removed net N$108: Q93.S, Q94.D
- removed net N$109: Q94.S, Q95.D
- removed net N$11: Q11.S, Q12.D
- removed net N$110: Q96.S, Q97.D
- removed net N$111: Q105.G, Q106.D, Q92.G, Q98.G, R46.1
- removed net N$112: Q97.S, Q98.D
- removed net N$113: Q96.G, Q99.D, R43.1
- removed net N$114: Q100.D, Q99.S
- removed net N$115: Q101.S, Q102.D
- removed net N$116: O4.S, Q101.D, Q103.G, R44.1
- removed net N$117: Q102.G, Q103.D, R45.1
- removed net N$118: Q103.S, Q104.D
- removed net N$119: Q104.S, Q105.D
- removed net N$14: Q18.G, Q24.D, Q28.G, Q29.G, R10.1
- removed net N$141: Q126.G, Q129.D, Q140.G, R57.1
- removed net N$142: Q126.D, Q131.G, Q135.G, R56.1
- removed net N$143: I2.S, Q127.G
- removed net N$144: Q126.S, Q127.D
- removed net N$145: Q127.S, Q128.D
- removed net N$146: Q129.G, Q132.D, Q136.G, Q137.G, R58.1
- removed net N$148: Q129.S, Q130.D
- removed net N$149: Q130.S, Q131.D
- removed net N$150: Q132.S, Q133.D
- removed net N$151: Q128.G, Q134.G, Q141.G, Q142.D, R62.1
- removed net N$152: Q133.S, Q134.D
- removed net N$153: Q132.G, Q135.D, R59.1
- removed net N$154: Q135.S, Q136.D
- removed net N$155: Q137.S, Q138.D
- removed net N$156: O2.S, Q137.D, Q139.G, R60.1
- removed net N$157: Q138.G, Q139.D, R61.1
- removed net N$158: Q139.S, Q140.D
- removed net N$159: Q140.S, Q141.D
- removed net N$181: Q162.G, Q165.D, Q176.G, R73.1
- removed net N$182: Q162.D, Q167.G, Q171.G, R72.1
- removed net N$183: I1.S, Q163.G
- removed net N$184: Q162.S, Q163.D
- removed net N$185: Q163.S, Q164.D
- removed net N$186: Q165.G, Q168.D, Q172.G, Q173.G, R74.1
- removed net N$188: Q165.S, Q166.D
- removed net N$189: Q166.S, Q167.D
- removed net N$190: Q168.S, Q169.D
- removed net N$191: Q164.G, Q170.G, Q177.G, Q178.D, R78.1
- removed net N$192: Q169.S, Q170.D
- removed net N$193: Q168.G, Q171.D, R75.1
- removed net N$194: Q171.S, Q172.D
- removed net N$195: Q173.S, Q174.D
- removed net N$196: O1.S, Q173.D, Q175.G, R76.1
- removed net N$197: Q174.G, Q175.D, R77.1
- removed net N$198: Q175.S, Q176.D
- removed net N$199: Q176.S, Q177.D
- removed net N$22: Q24.S, Q25.D
- removed net N$221: Q198.G, Q201.D, Q212.G, R89.1
- removed net N$222: Q198.D, Q203.G, Q207.G, R88.1
- removed net N$223: I0.S, Q199.G
- removed net N$224: Q198.S, Q199.D
- removed net N$225: Q199.S, Q200.D
- removed net N$226: Q201.G, Q204.D, Q208.G, Q209.G, R90.1
- removed net N$228: Q201.S, Q202.D
- removed net N$229: Q202.S, Q203.D
- removed net N$230: Q204.S, Q205.D
- removed net N$231: Q200.G, Q206.G, Q213.G, Q214.D, R94.1
- removed net N$232: Q205.S, Q206.D
- removed net N$233: Q204.G, Q207.D, R91.1
- removed net N$234: Q207.S, Q208.D
- removed net N$235: Q209.S, Q210.D
- removed net N$236: O0.S, Q209.D, Q211.G, R92.1
- removed net N$237: Q210.G, Q211.D, R93.1
- removed net N$238: Q211.S, Q212.D
- removed net N$239: Q212.S, Q213.D
- removed net N$41: Q36.G, Q39.D, Q50.G, R17.1
- removed net N$42: Q36.D, Q41.G, Q45.G, R16.1
- removed net N$43: I5.S, Q37.G
- removed net N$44: Q36.S, Q37.D
- removed net N$45: Q37.S, Q38.D
- removed net N$46: Q39.G, Q42.D, Q46.G, Q47.G, R18.1
- removed net N$48: Q39.S, Q40.D
- removed net N$49: Q40.S, Q41.D
- removed net N$50: Q42.S, Q43.D
- removed net N$51: Q38.G, Q44.G, Q51.G, Q52.D, R22.1
- removed net N$52: Q43.S, Q44.D
- removed net N$53: Q42.G, Q45.D, R19.1
- removed net N$54: Q45.S, Q46.D
- removed net N$55: Q47.S, Q48.D
- removed net N$56: O5.S, Q47.D, Q49.G, R20.1
- removed net N$57: Q48.G, Q49.D, R21.1
- removed net N$58: Q49.S, Q50.D
- removed net N$59: Q50.S, Q51.D
- removed net N$61: Q54.G, Q57.D, Q68.G, R25.1
- removed net N$62: Q54.D, Q59.G, Q63.G, R24.1
- removed net N$63: I6.S, Q55.G
- removed net N$64: Q54.S, Q55.D
- removed net N$65: Q55.S, Q56.D
- removed net N$66: Q57.G, Q60.D, Q64.G, Q65.G, R26.1
- removed net N$68: Q57.S, Q58.D
- removed net N$69: Q58.S, Q59.D
- removed net N$70: Q60.S, Q61.D
- removed net N$71: Q56.G, Q62.G, Q69.G, Q70.D, R30.1
- removed net N$72: Q61.S, Q62.D
- removed net N$73: Q60.G, Q63.D, R27.1
- removed net N$74: Q63.S, Q64.D
- removed net N$75: Q65.S, Q66.D
- removed net N$76: O6.S, Q65.D, Q67.G, R28.1
- removed net N$77: Q66.G, Q67.D, R29.1
- removed net N$78: Q67.S, Q68.D
- removed net N$79: Q68.S, Q69.D
- removed net N$81: Q72.G, Q75.D, Q86.G, R33.1
- removed net N$82: Q72.D, Q77.G, Q81.G, R32.1
- removed net N$83: I3.S, Q73.G
- removed net N$84: Q72.S, Q73.D
- removed net N$85: Q73.S, Q74.D
- removed net N$86: Q75.G, Q78.D, Q82.G, Q83.G, R34.1
- removed net N$88: Q75.S, Q76.D
- removed net N$89: Q76.S, Q77.D
- removed net N$90: Q78.S, Q79.D
- removed net N$91: Q74.G, Q80.G, Q87.G, Q88.D, R38.1
- removed net N$92: Q79.S, Q80.D
- removed net N$93: Q78.G, Q81.D, R35.1
- removed net N$94: Q81.S, Q82.D
- removed net N$95: Q83.S, Q84.D
- removed net N$96: O3.S, Q83.D, Q85.G, R36.1
- removed net N$97: Q84.G, Q85.D, R37.1
- removed net N$98: Q85.S, Q86.D
- removed net N$99: Q86.S, Q87.D
- new net N$12: O1.S, Q11.D, R5.1
- new net N$15: I5.S, Q13.G
- new net N$16: Q13.D, Q14.D, Q18.G, R7.1
- new net N$2: Q1.D, Q11.G, Q2.D, R1.1
- new net N$20: Q16.G, Q17.G, SEL2.S
- new net N$28: Q20.S, Q22.D
- new net N$29: Q22.G, Q23.G, SEL3.S
- new net N$30: I8.S, Q20.G
- new net N$34: Q25.D, Q26.D, Q30.G, R13.1
- new net N$37: Q28.G, Q29.G, SEL4.S
- new net N$38: I10.S, Q26.G
- new net N$39: Q27.G, Q29.D, R14.1
- new net N$40: O4.S, Q30.D, R15.1
- new net N$5: Q4.G, Q9.G, SEL1.S
- new net N$6: I4.S, Q2.G
- new net N$7: Q3.G, Q9.D, R3.1
- net GND: now also Q11.S, Q15.S, Q16.S, Q17.S, Q18.S, Q21.S, Q22.S, Q23.S, Q24.S, Q27.S, Q29.S, Q3.S, Q4.S, Q9.S; no longer Q100.S, Q102.S, Q105.S, Q106.S, Q12.S, Q128.S, Q131.S, Q134.S, Q136.S, Q138.S, Q141.S, Q142.S, Q164.S, Q167.S, Q170.S, Q172.S, Q174.S, Q177.S, Q178.S, Q20.S, Q200.S, Q203.S, Q206.S, Q208.S, Q210.S, Q213.S, Q214.S, Q26.S, Q33.S, Q34.S, Q38.S, Q41.S, Q44.S, Q46.S, Q48.S, Q51.S, Q52.S, Q56.S, Q59.S, Q62.S, Q64.S, Q66.S, Q69.S, Q70.S, Q74.S, Q77.S, Q80.S, Q82.S, Q84.S, Q87.S, Q88.S, Q92.S, Q95.S, Q98.S
- net N$1: now also I3.S, Q1.G; no longer Q18.D, Q2.G, Q32.G, R8.1
- net N$17: now also Q13.S, Q15.D; no longer CLK.S, Q130.G, Q133.G, Q166.G, Q169.G, Q19.G, Q202.G, Q205.G, Q25.G, Q40.G, Q43.G, Q58.G, Q61.G, Q76.G, Q79.G, Q94.G, Q97.G
- net N$19: now also Q14.S, Q16.D; no longer Q18.S, Q19.D
- net N$21: now also I6.S, Q14.G; no longer Q19.S, Q20.D
- net N$23: now also Q15.G, Q17.D, R8.1; no longer Q12.G, Q26.G, Q33.G, Q34.D, R14.1
- net N$24: now also O2.S, Q18.D, R9.1; no longer Q25.S, Q26.D
- net N$25: now also I7.S, Q19.G; no longer Q24.G, Q27.D, R11.1
- net N$26: now also Q19.D, Q20.D, Q24.G, R10.1; no longer Q27.S, Q28.D
- net N$27: now also Q19.S, Q21.D; no longer Q29.S, Q30.D
- net N$3: now also Q1.S, Q3.D; no longer Q2.D, Q20.G, Q27.G, R1.1
- net N$31: now also Q21.G, Q23.D, R11.1; no longer O7.S, Q29.D, Q31.G, R12.1
- net N$32: now also O3.S, Q24.D, R12.1; no longer Q30.G, Q31.D, R13.1
- net N$33: now also I9.S, Q25.G; no longer Q31.S, Q32.D
- net N$35: now also Q25.S, Q27.D; no longer Q32.S, Q33.D
- net N$36: now also Q26.S, Q28.D; no longer Q106.G, Q142.G, Q178.G, Q214.G, Q34.G, Q52.G, Q70.G, Q88.G, R.S
- net N$4: now also Q2.S, Q4.D; no longer I7.S, Q11.G
- net VCC: now also R15.2, R3.2, R5.2, R7.2, R9.2; no longer R16.2, R17.2, R18.2, R19.2, R20.2, R21.2, R22.2, R24.2, R25.2, R26.2, R27.2, R28.2, R29.2, R30.2, R32.2, R33.2, R34.2, R35.2, R36.2, R37.2, R38.2, R40.2, R41.2, R42.2, R43.2, R44.2, R45.2, R46.2, R56.2, R57.2, R58.2, R59.2, R60.2, R61.2, R62.2, R72.2, R73.2, R74.2, R75.2, R76.2, R77.2, R78.2, R88.2, R89.2, R90.2, R91.2, R92.2, R93.2, R94.2
Other:
- note added: "AOI2x2"
- note added: "MUX"
- note removed: "BYTE"
- note removed: "DFF"
- note removed: "NAND"
- note removed: "NAND3"
- moved on the sheet: I3, I4, I5, I6, I7, O1, O2, O3, O4, Q11, Q18, Q19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

Commit message: Optimized reset and mux with inversions
No single not gates
Parts:
- removed I10, I3, I4, I5, I6, I7, I8, I9, O1, O2, O3, O4, SEL1, SEL2, SEL3, SEL4: TPPAD6, ellajameson-core:TPPAD6
- removed Q1, Q11, Q13, Q14, Q15, Q16, Q17, Q18, Q19, Q2, Q20, Q21, Q22, Q23, Q24, Q25, Q26, Q27, Q28, Q29, Q3, Q30, Q4, Q9: 2N7002, ellajameson-core:2N7002
- removed R1, R10, R11, R12, R13, R14, R15, R3, R5, R7, R8, R9: (no value), ellajameson-core:RES0603
- added U1: SN74S374N, ellajameson-core:SN74S374N
Connections:
- removed net N$1: I3.S, Q1.G
- removed net N$12: O1.S, Q11.D, R5.1
- removed net N$15: I5.S, Q13.G
- removed net N$16: Q13.D, Q14.D, Q18.G, R7.1
- removed net N$17: Q13.S, Q15.D
- removed net N$19: Q14.S, Q16.D
- removed net N$2: Q1.D, Q11.G, Q2.D, R1.1
- removed net N$20: Q16.G, Q17.G, SEL2.S
- removed net N$21: I6.S, Q14.G
- removed net N$23: Q15.G, Q17.D, R8.1
- removed net N$24: O2.S, Q18.D, R9.1
- removed net N$25: I7.S, Q19.G
- removed net N$26: Q19.D, Q20.D, Q24.G, R10.1
- removed net N$27: Q19.S, Q21.D
- removed net N$28: Q20.S, Q22.D
- removed net N$29: Q22.G, Q23.G, SEL3.S
- removed net N$3: Q1.S, Q3.D
- removed net N$30: I8.S, Q20.G
- removed net N$31: Q21.G, Q23.D, R11.1
- removed net N$32: O3.S, Q24.D, R12.1
- removed net N$33: I9.S, Q25.G
- removed net N$34: Q25.D, Q26.D, Q30.G, R13.1
- removed net N$35: Q25.S, Q27.D
- removed net N$36: Q26.S, Q28.D
- removed net N$37: Q28.G, Q29.G, SEL4.S
- removed net N$38: I10.S, Q26.G
- removed net N$39: Q27.G, Q29.D, R14.1
- removed net N$4: Q2.S, Q4.D
- removed net N$40: O4.S, Q30.D, R15.1
- removed net N$5: Q4.G, Q9.G, SEL1.S
- removed net N$6: I4.S, Q2.G
- removed net N$7: Q3.G, Q9.D, R3.1
- net GND: now also U1.GND; no longer Q11.S, Q15.S, Q16.S, Q17.S, Q18.S, Q21.S, Q22.S, Q23.S, Q24.S, Q27.S, Q28.S, Q29.S, Q3.S, Q30.S, Q4.S, Q9.S
- net VCC: now also U1.VCC; no longer R1.2, R10.2, R11.2, R12.2, R13.2, R14.2, R15.2, R3.2, R5.2, R7.2, R8.2, R9.2
Other:
- note removed: "AOI2x2"
- note removed: "MUX"
- note removed: "NOT"
