File: Eagle/PCBs/Counter Toy/BLOCKS.sch (EAGLE design)
At the start: 4 parts, among them Q1 2N7002

Commit message: Wow, 92 transistors and 8 LEDs
Parts:
- removed D1: (no value), ellajameson-core:LED0603
- removed LED1: TPTHT, ellajameson-core:TPTHT
- added DRAINA1, DRAINA10, DRAINA11, DRAINA12, DRAINA13, DRAINA14, DRAINA15, DRAINA16, DRAINA17, DRAINA18, DRAINA19, DRAINA20, DRAINA6, DRAINA7, DRAINA8, DRAINA9, DRAINB1, DRAINB10, DRAINB11, DRAINB12, DRAINB13, DRAINB14, DRAINB15, DRAINB16, DRAINB17, DRAINB18, DRAINB19, DRAINB20, DRAINB6, DRAINB7, DRAINB8, DRAINB9, GATEA1, GATEA10, GATEA11, GATEA12, GATEA13, GATEA14, GATEA15, GATEA16, GATEA17, GATEA18, GATEA19, GATEA20, GATEA6, GATEA7, GATEA8, GATEA9, GATEB1, GATEB10, GATEB11, GATEB12, GATEB13, GATEB14, GATEB15, GATEB16, GATEB17, GATEB18, GATEB19, GATEB20, GATEB6, GATEB7, GATEB8, GATEB9, SOURCEA1, SOURCEA10, SOURCEA11, SOURCEA12, SOURCEA13, SOURCEA14, SOURCEA15, SOURCEA16, SOURCEA17, SOURCEA18, SOURCEA19, SOURCEA20, SOURCEA6, SOURCEA7, SOURCEA8, SOURCEA9, SOURCEB1, SOURCEB10, SOURCEB11, SOURCEB12, SOURCEB13, SOURCEB14, SOURCEB15, SOURCEB16, SOURCEB17, SOURCEB18, SOURCEB19, SOURCEB20, SOURCEB6, SOURCEB7, SOURCEB8, SOURCEB9: TPTHT, ellajameson-core:TPTHT
- added JD1, JD10, JD11, JD12, JD13, JD14, JD15, JD16, JD17, JD18, JD19, JD20, JD6, JD7, JD8, JD9, JN1, JN10, JN11, JN12, JN13, JN14, JN15, JN16, JN17, JN18, JN19, JN20, JN6, JN7, JN8, JN9, JP1, JP10, JP11, JP12, JP13, JP14, JP15, JP16, JP17, JP18, JP19, JP20, JP6, JP7, JP8, JP9, JS1, JS10, JS11, JS12, JS13, JS14, JS15, JS16, JS17, JS18, JS19, JS20, JS6, JS7, JS8, JS9: SJ_NO_THIN, ellajameson-core:SJ_NO_THIN
- added Q10, Q11, Q12, Q13, Q14, Q15, Q16, Q17, Q18, Q19, Q20, Q6, Q7, Q8, Q9: 2N7002, ellajameson-core:2N7002
- added R10, R11, R12, R13, R14, R15, R16, R17, R18, R19, R20, R6, R7, R8, R9: 10k, ellajameson-core:RES0603
- R1: value 330 -> 10k
Connections:
- removed net N$8: LED1.S, Q1.G
- new net N$2: JN9.2, JS9.2, Q1.S, SOURCEA9.S, SOURCEB9.S
- new net N$21: JN1.2, JS1.2, Q6.S, SOURCEA1.S, SOURCEB1.S
- new net N$22: DRAINA1.S, DRAINB1.S, JD1.2, JP1.1, Q6.D
- new net N$23: GATEA1.S, GATEB1.S, Q6.G
- new net N$24: JP6.2, R7.1
- new net N$25: JN6.2, JS6.2, Q7.S, SOURCEA6.S, SOURCEB6.S
- new net N$26: DRAINA6.S, DRAINB6.S, JD1.1, JD6.2, JP6.1, Q7.D
- new net N$27: GATEA6.S, GATEB6.S, Q7.G
- new net N$28: JP7.2, R8.1
- new net N$29: JN7.2, JS7.2, Q8.S, SOURCEA7.S, SOURCEB7.S
- new net N$30: DRAINA7.S, DRAINB7.S, JD6.1, JD7.2, JP7.1, Q8.D
- new net N$31: GATEA7.S, GATEB7.S, Q8.G
- new net N$32: JP8.2, R9.1
- new net N$33: JN8.2, JS8.2, Q9.S, SOURCEA8.S, SOURCEB8.S
- new net N$34: DRAINA8.S, DRAINB8.S, JD7.1, JD8.2, JP8.1, Q9.D
- new net N$35: GATEA8.S, GATEB8.S, Q9.G
- new net N$36: GATEA9.S, GATEB9.S, Q1.G
- new net N$37: JP10.2, R10.1
- new net N$38: JN10.2, JS10.2, Q10.S, SOURCEA10.S, SOURCEB10.S
- new net N$39: DRAINA10.S, DRAINB10.S, JD10.2, JD9.1, JP10.1, Q10.D
- new net N$40: GATEA10.S, GATEB10.S, Q10.G
- new net N$41: JP11.2, R11.1
- new net N$42: JN11.2, JS11.2, Q11.S, SOURCEA11.S, SOURCEB11.S
- new net N$43: DRAINA11.S, DRAINB11.S, JD10.1, JD11.2, JP11.1, Q11.D
- new net N$44: GATEA11.S, GATEB11.S, Q11.G
- new net N$45: JP12.2, R12.1
- new net N$46: JN12.2, JS12.2, Q12.S, SOURCEA12.S, SOURCEB12.S
- new net N$47: DRAINA12.S, DRAINB12.S, JD11.1, JD12.2, JP12.1, Q12.D
- new net N$48: GATEA12.S, GATEB12.S, Q12.G
- new net N$49: JP13.2, R13.1
- new net N$50: JN13.2, JS13.2, Q13.S, SOURCEA13.S, SOURCEB13.S
- new net N$51: DRAINA13.S, DRAINB13.S, JD12.1, JD13.2, JP13.1, Q13.D
- new net N$52: GATEA13.S, GATEB13.S, Q13.G
- new net N$53: JP14.2, R14.1
- new net N$54: JN14.2, JS14.2, Q14.S, SOURCEA14.S, SOURCEB14.S
- new net N$55: DRAINA14.S, DRAINB14.S, JD13.1, JD14.2, JP14.1, Q14.D
- new net N$56: GATEA14.S, GATEB14.S, Q14.G
- new net N$57: JP15.2, R15.1
- new net N$58: JN15.2, JS15.2, Q15.S, SOURCEA15.S, SOURCEB15.S
- new net N$59: DRAINA15.S, DRAINB15.S, JD14.1, JD15.2, JP15.1, Q15.D
- new net N$60: GATEA15.S, GATEB15.S, Q15.G
- new net N$61: JP16.2, R16.1
- new net N$62: JN16.2, JS16.2, Q16.S, SOURCEA16.S, SOURCEB16.S
- new net N$63: DRAINA16.S, DRAINB16.S, JD15.1, JD16.2, JP16.1, Q16.D
- new net N$64: GATEA16.S, GATEB16.S, Q16.G
- new net N$65: JP17.2, R17.1
- new net N$66: JN17.2, JS17.2, Q17.S, SOURCEA17.S, SOURCEB17.S
- new net N$67: DRAINA17.S, DRAINB17.S, JD16.1, JD17.2, JP17.1, Q17.D
- new net N$68: GATEA17.S, GATEB17.S, Q17.G
- new net N$69: JP18.2, R18.1
- new net N$7: JP1.2, R6.1
- new net N$70: JN18.2, JS18.2, Q18.S, SOURCEA18.S, SOURCEB18.S
- new net N$71: DRAINA18.S, DRAINB18.S, JD17.1, JD18.2, JP18.1, Q18.D
- new net N$72: GATEA18.S, GATEB18.S, Q18.G
- new net N$73: JP19.2, R19.1
- new net N$74: JN19.2, JS19.2, Q19.S, SOURCEA19.S, SOURCEB19.S
- new net N$75: DRAINA19.S, DRAINB19.S, JD18.1, JD19.2, JP19.1, Q19.D
- new net N$76: GATEA19.S, GATEB19.S, Q19.G
- new net N$77: JP20.2, R20.1
- new net N$78: JN20.2, JS20.2, Q20.S, SOURCEA20.S, SOURCEB20.S
- new net N$79: DRAINA20.S, DRAINB20.S, JD19.1, JD20.2, JP20.1, Q20.D
- new net N$80: GATEA20.S, GATEB20.S, Q20.G
- net GND: now also JN1.1, JN10.1, JN11.1, JN12.1, JN13.1, JN14.1, JN15.1, JN16.1, JN17.1, JN18.1, JN19.1, JN20.1, JN6.1, JN7.1, JN8.1, JN9.1; no longer Q1.S
- net N$1: now also JP9.2, R1.1; no longer D1.K, Q1.D
- net N$5: now also DRAINA9.S, DRAINB9.S, JD8.1, JD9.2, JP9.1, Q1.D; no longer D1.A, R1.1
- net VCC: now also R10.2, R11.2, R12.2, R13.2, R14.2, R15.2, R16.2, R17.2, R18.2, R19.2, R20.2, R6.2, R7.2, R8.2, R9.2
Other:
- note added: "NMOS Logic Transistor Cell"
- note removed: "LED Output"
- moved on the sheet: Q1, R1
