File: Eagle/PCBs/NMOS Experimenter Board/experimenter.brd (EAGLE design)
At the start: 16 parts, among them Q1 2N7002

Commit message: Testing open collector setup
Parts:
- removed D1: (no value), ellajameson-core:CHIP-LED0603
- removed DRAINA1, DRAINB1, DRAINC1, DRAIND1, GATE1, SOURCEA1, SOURCEB1, SOURCEC1, SOURCED1: TPWIRE, ellajameson-core:TP_TH_WIRE
- removed JD1, JN1, JP1, JS1: SJ_NO, ellajameson-core:SJ_2S-NO
- removed Q1: 2N7002, ellajameson-core:SOT23
- removed R1: (no value), ellajameson-core:R0603
Connections:
- removed net GND: JN1.1
- removed net N$5: D1.A, JP1.2, R1.1
- removed net N$6: D1.C, DRAINA1.TP, DRAINB1.TP, DRAINC1.TP, DRAIND1.TP, JD1.2, JP1.1, Q1.3
- removed net N$7: JN1.2, JS1.2, Q1.2, SOURCEA1.TP, SOURCEB1.TP, SOURCEC1.TP, SOURCED1.TP
- removed net N$8: GATE1.TP, Q1.1
- removed net VCC: R1.2
Routing:
- net N$6: track 11.0 -> 0.00 mm
- net N$7: track 9.49 -> 0.00 mm
- net N$5: track 3.87 -> 0.00 mm
- net GND: track 3.07 -> 0.00 mm, vias 1 -> 0
- net N$8: track 1.97 -> 0.00 mm
- net VCC: track 1.26 -> 0.00 mm, vias 1 -> 0
Other:
- board text removed: "#X"
- board text removed: "D"
- board text removed: "G"
- board text removed: "S"
Changed lines of the file:
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@@
 <board>
 <plain>
-<text x="0.254" y="1.651" size="0.8128" layer="22">G</text>
-<text x="4.572" y="10.16" size="0.8128" layer="21">D</text>
-<text x="4.699" y="2.794" size="0.8128" layer="21">S</text>
-<wire x1="0" y1="0" x2="0" y2="13.335" width="0.1524" layer="21"/>
-<wire x1="0" y1="13.335" x2="5.588" y2="13.335" width="0.1524" layer="21"/>
-<wire x1="5.588" y1="0" x2="0" y2="0" width="0.1524" layer="21"/>
-<wire x1="5.588" y1="0" x2="5.588" y2="13.335" width="0.1524" layer="21"/>
-<wire x1="0" y1="0" x2="0" y2="13.335" width="0.1524" layer="22"/>
-<wire x1="0" y1="13.335" x2="5.588" y2="13.335" width="0.1524" layer="22"/>
-<wire x1="5.588" y1="0" x2="0" y2="0" width="0.1524" layer="22"/>
-<wire x1="5.588" y1="0" x2="5.588" y2="13.335" width="0.1524" layer="22"/>
-<text x="0.254" y="1.651" size="0.8128" layer="21" rot="MR0" align="bottom-right">G</text>
-<text x="4.699" y="2.794" size="0.8128" layer="22" rot="MR0" align="bottom-right">S</text>
-<text x="4.572" y="10.16" size="0.8128" layer="22" rot="MR0" align="bottom-right">D</text>
-<text x="5.461" y="13.208" size="0.8128" layer="21" rot="R270" align="top-left">#X</text>
-<text x="5.461" y="13.208" size="0.8128" layer="22" rot="MR90" align="top-right">#X</text>
 </plain>
 <attributes>
@@
 </autorouter>
 <elements>
-<element name="Q1" library="ellajameson-core" library_urn="urn:adsk.eagle:library:3740209" package="SOT23" package3d_urn="urn:adsk.eagle:package:7587823/4" value="2N7002" x="1.651" y="6.35" smashed="yes"/>
-<element name="R1" library="ellajameson-core" library_urn="urn:adsk.eagle:library:3740209" package="R0603" package3d_urn="urn:adsk.eagle:package:7587835/4" value="" x="1.778" y="11.811" smashed="yes"/>
-<element name="JP1" library="ellajameson-core" library_urn="urn:adsk.eagle:library:3740209" package="SJ_2S-NO" package3d_urn="urn:adsk.eagle:package:26612370/2" value="SJ_NO" x="1.016" y="9.398" smashed="yes" rot="R90"/>
-<element name="D1" library="ellajameson-core" library_urn="urn:adsk.eagle:library:3740209" package="CHIP-LED0603" package3d_urn="urn:adsk.eagle:package:7587825/3" value="" x="2.794" y="9.525" smashed="yes" rot="R180"/>
-<element name="JN1" library="ellajameson-core" library_urn="urn:adsk.eagle:library:3740209" package="SJ_2S-NO" package3d_urn="urn:adsk.eagle:package:26612370/2" value="SJ_NO" x="2.413" y="3.302" smashed="yes"/>
-<element name="GATE1" library="ellajameson-core" library_urn="urn:adsk.eagle:library:3740209" package="TP_TH_WIRE" package3d_urn="urn:adsk.eagle:package:40139460/1" value="TPWIRE" x="0.762" y="3.302" smashed="yes"/>
-<element name="DRAINA1" library="ellajameson-core" library_urn="urn:adsk.eagle:library:3740209" package="TP_TH_WIRE" package3d_urn="urn:adsk.eagle:package:40139460/1" value="TPWIRE" x="3.937" y="12.446" smashed="yes"/>
-<element name="SOURCEA1" library="ellajameson-core" library_urn="urn:adsk.eagle:library:3740209" package="TP_TH_WIRE" package3d_urn="urn:adsk.eagle:package:40139460/1" value="TPWIRE" x="4.064" y="5.08" smashed="yes"/>
-<element name="JS1" library="ellajameson-core" library_urn="urn:adsk.eagle:library:3740209" package="SJ_2S-NO" package3d_urn="urn:adsk.eagle:package:26612370/2" value="SJ_NO" x="2.286" y="1.143" smashed="yes" rot="R90"/>
-<element name="JD1" library="ellajameson-core" library_urn="urn:adsk.eagle:library:3740209" package="SJ_2S-NO" package3d_urn="urn:adsk.eagle:package:26612370/2" value="SJ_NO" x="4.445" y="6.858" smashed="yes" rot="R180"/>
-<element name="DRAINB1" library="ellajameson-core" library_urn="urn:adsk.eagle:library:3740209" package="TP_TH_WIRE" package3d_urn="urn:adsk.eagle:package:40139460/1" value="TPWIRE" x="3.937" y="11.176" smashed="yes"/>
-<element name="DRAINC1" library="ellajameson-core" library_urn="urn:adsk.eagle:library:3740209" package="TP_TH_WIRE" package3d_urn="urn:adsk.eagle:package:40139460/1" value="TPWIRE" x="3.937" y="9.906" smashed="yes"/>
-<element name="DRAIND1" library="ellajameson-core" library_urn="urn:adsk.eagle:library:3740209" package="TP_TH_WIRE" package3d_urn="urn:adsk.eagle:package:40139460/1" value="TPWIRE" x="3.937" y="8.636" smashed="yes"/>
-<element name="SOURCEB1" library="ellajameson-core" library_urn="urn:adsk.eagle:library:3740209" package="TP_TH_WIRE" package3d_urn="urn:adsk.eagle:package:40139460/1" value="TPWIRE" x="4.064" y="3.81" smashed="yes"/>
-<element name="SOURCEC1" library="ellajameson-core" library_urn="urn:adsk.eagle:library:3740209" package="TP_TH_WIRE" package3d_urn="urn:adsk.eagle:package:40139460/1" value="TPWIRE" x="4.064" y="2.54" smashed="yes"/>
-<element name="SOURCED1" library="ellajameson-core" library_urn="urn:adsk.eagle:library:3740209" package="TP_TH_WIRE" package3d_urn="urn:adsk.eagle:package:40139460/1" value="TPWIRE" x="4.064" y="1.27" smashed="yes"/>
 </elements>
 <signals>
-<signal name="VCC">
-<contactref element="R1" pad="2"/>
-<wire x1="2.628" y1="11.811" x2="2.628" y2="12.661" width="0.3048" layer="1"/>
-<wire x1="2.628" y1="12.661" x2="2.921" y2="12.954" width="0.3048" layer="1"/>
-<via x="2.921" y="12.954" extent="1-16" drill="0.35"/>
-</signal>
-<signal name="N$5">
-<contactref element="R1" pad="1"/>
-<contactref element="D1" pad="A"/>
-<contactref element="JP1" pad="2"/>
-<wire x1="1.016" y1="9.906" x2="2.425" y2="9.906" width="0.3048" layer="1"/>
-<wire x1="2.425" y1="9.906" x2="2.794" y2="10.275" width="0.3048" layer="1"/>
-<wire x1="1.016" y1="9.906" x2="1.016" y2="11.723" width="0.3048" layer="1"/>
-<wire x1="1.016" y1="11.723" x2="0.928" y2="11.811" width="0.3048" layer="1"/>
-</signal>
-<signal name="N$6">
-<contactref element="JP1" pad="1"/>
-<contactref element="D1" pad="C"/>
-<contactref element="Q1" pad="3"/>
-<contactref element="DRAINA1" pad="TP"/>
-<contactref element="JD1" pad="2"/>
-<wire x1="1.016" y1="8.89" x2="1.143" y2="8.89" width="0.3048" layer="1"/>
-<wire x1="1.143" y1="8.89" x2="2.679" y2="8.89" width="0.3048" layer="1"/>
-<wire x1="2.679" y1="8.89" x2="2.794" y2="8.775" width="0.3048" layer="1"/>
-<contactref element="DRAINB1" pad="TP"/>
-<contactref element="DRAINC1" pad="TP"/>
-<contactref element="DRAIND1" pad="TP"/>
-<wire x1="1.651" y1="7.45" x2="1.143" y2="7.958" width="0.3048" layer="1"/>
-<wire x1="1.143" y1="7.958" x2="1.143" y2="8.89" width="0.3048" layer="1"/>
-<wire x1="2.794" y1="8.775" x2="2.933" y2="8.636" width="0.3048" layer="1"/>
-<wire x1="2.933" y1="8.636" x2="3.937" y2="8.636" width="0.3048" layer="1"/>
-<wire x1="3.937" y1="9.906" x2="3.937" y2="8.636" width="0.3048" layer="1"/>
-<wire x1="3.937" y1="12.446" x2="3.937" y2="11.176" width="0.3048" layer="1"/>
-<wire x1="3.937" y1="11.176" x2="3.937" y2="9.906" width="0.3048" layer="1"/>
-<wire x1="1.651" y1="7.45" x2="2.583" y2="7.45" width="0.3048" layer="1"/>
-<wire x1="3.175" y1="6.858" x2="3.937" y2="6.858" width="0.3048" layer="1"/>
-<wire x1="2.583" y1="7.45" x2="3.175" y2="6.858" width="0.3048" layer="1"/>
-</signal>
-<signal name="N$7">
-<contactref element="JN1" pad="2"/>
-<contactref element="Q1" pad="2"/>
-<contactref element="SOURCEA1" pad="TP"/>
-<contactref element="JS1" pad="2"/>
-<contactref element="SOURCEB1" pad="TP"/>
-<contactref element="SOURCEC1" pad="TP"/>
-<contactref element="SOURCED1" pad="TP"/>
-<wire x1="2.601" y1="5.25" x2="2.921" y2="4.93" width="0.3048" layer="1"/>
-<wire x1="2.921" y1="4.93" x2="2.921" y2="3.302" width="0.3048" layer="1"/>
-<wire x1="2.286" y1="1.651" x2="2.54" y2="1.651" width="0.3048" layer="1"/>
-<wire x1="2.54" y1="1.651" x2="2.921" y2="2.032" width="0.3048" layer="1"/>
-<wire x1="2.921" y1="2.032" x2="2.921" y2="3.302" width="0.3048" layer="1"/>
-<wire x1="2.601" y1="5.25" x2="3.894" y2="5.25" width="0.3048" layer="1"/>
-<wire x1="3.894" y1="5.25" x2="4.064" y2="5.08" width="0.3048" layer="1"/>
-<wire x1="4.064" y1="5.08" x2="4.064" y2="3.81" width="0.3048" layer="1"/>
-<wire x1="4.064" y1="3.81" x2="4.064" y2="2.54" width="0.3048" layer="1"/>
-<wire x1="4.064" y1="2.54" x2="4.064" y2="1.27" width="0.3048" layer="1"/>
-</signal>
-<signal name="GND">
-<contactref element="JN1" pad="1"/>
-<wire x1="1.905" y1="3.302" x2="1.905" y2="2.921" width="0.3048" layer="1"/>
-<wire x1="1.905" y1="2.921" x2="1.27" y2="2.286" width="0.3048" layer="1"/>
-<wire x1="1.27" y1="2.286" x2="1.27" y2="1.397" width="0.3048" layer="1"/>
-<wire x1="1.27" y1="1.397" x2="0.635" y2="0.762" width="0.3048" layer="1"/>
-<via x="0.635" y="0.762" extent="1-16" drill="0.35"/>
-</signal>
-<signal name="N$8">
-<contactref element="Q1" pad="1"/>
-<contactref element="GATE1" pad="TP"/>
-<wire x1="0.701" y1="5.25" x2="0.762" y2="5.189" width="0.3048" layer="1"/>
-<wire x1="0.762" y1="5.189" x2="0.762" y2="3.302" width="0.3048" layer="1"/>
-</signal>
 </signals>
 <mfgpreviewcolors>
@@
 </board>
 </drawing>
-<compatibility>
-<note version="8.2" severity="warning">
-Since Version 8.2, EAGLE supports online libraries. The ids
-of those online libraries will not be understood (or retained)
-with this version.
-</note>
-<note version="8.3" severity="warning">
-Since Version 8.3, EAGLE supports URNs for individual library
-assets (packages, symbols, and devices). The URNs of those assets
-will not be understood (or retained) with this version.
-</note>
-<note version="8.3" severity="warning">
-Since Version 8.3, EAGLE supports the association of 3D packages
-with devices in libraries, schematics, and board files. Those 3D
-packages will not be understood (or retained) with this version.
-</note>
-</compatibility>
 </eagle>

Commit message: Update packages
Parts:
- added D10, D11, D12, D13, D14, D15, D16, D17, D18, D19, D2, D20, D21, D22, D23, D24, D25, D3, D4, D5, D6, D7, D8, D9: (no value), ellajameson-core:CHIP-LED0603
- added DRAINA10, DRAINA11, DRAINA12, DRAINA13, DRAINA14, DRAINA15, DRAINA16, DRAINA17, DRAINA18, DRAINA19, DRAINA2, DRAINA20, DRAINA21, DRAINA22, DRAINA23, DRAINA24, DRAINA25, DRAINA3, DRAINA4, DRAINA5, DRAINA6, DRAINA7, DRAINA8, DRAINA9, DRAINB10, DRAINB11, DRAINB12, DRAINB13, DRAINB14, DRAINB15, DRAINB16, DRAINB17, DRAINB18, DRAINB19, DRAINB2, DRAINB20, DRAINB21, DRAINB22, DRAINB23, DRAINB24, DRAINB25, DRAINB3, DRAINB4, DRAINB5, DRAINB6, DRAINB7, DRAINB8, DRAINB9, DRAINC10, DRAINC11, DRAINC12, DRAINC13, DRAINC14, DRAINC15, DRAINC16, DRAINC17, DRAINC18, DRAINC19, DRAINC2, DRAINC20, DRAINC21, DRAINC22, DRAINC23, DRAINC24, DRAINC25, DRAINC3, DRAINC4, DRAINC5, DRAINC6, DRAINC7, DRAINC8, DRAINC9, DRAIND10, DRAIND11, DRAIND12, DRAIND13, DRAIND14, DRAIND15, DRAIND16, DRAIND17, DRAIND18, DRAIND19, DRAIND2, DRAIND20, DRAIND21, DRAIND22, DRAIND23, DRAIND24, DRAIND25, DRAIND3, DRAIND4, DRAIND5, DRAIND6, DRAIND7, DRAIND8, DRAIND9, GATE10, GATE11, GATE12, GATE13, GATE14, GATE15, GATE16, GATE17, GATE18, GATE19, GATE2, GATE20, GATE21, GATE22, GATE23, GATE24, GATE25, GATE3, GATE4, GATE5, GATE6, GATE7, GATE8, GATE9, SOURCEA10, SOURCEA11, SOURCEA12, SOURCEA13, SOURCEA14, SOURCEA15, SOURCEA16, SOURCEA17, SOURCEA18, SOURCEA19, SOURCEA2, SOURCEA20, SOURCEA21, SOURCEA22, SOURCEA23, SOURCEA24, SOURCEA25, SOURCEA3, SOURCEA4, SOURCEA5, SOURCEA6, SOURCEA7, SOURCEA8, SOURCEA9, SOURCEB10, SOURCEB11, SOURCEB12, SOURCEB13, SOURCEB14, SOURCEB15, SOURCEB16, SOURCEB17, SOURCEB18, SOURCEB19, SOURCEB2, SOURCEB20, SOURCEB21, SOURCEB22, SOURCEB23, SOURCEB24, SOURCEB25, SOURCEB3, SOURCEB4, SOURCEB5, SOURCEB6, SOURCEB7, SOURCEB8, SOURCEB9, SOURCEC10, SOURCEC11, SOURCEC12, SOURCEC13, SOURCEC14, SOURCEC15, SOURCEC16, SOURCEC17, SOURCEC18, SOURCEC19, SOURCEC2, SOURCEC20, SOURCEC21, SOURCEC22, SOURCEC23, SOURCEC24, SOURCEC25, SOURCEC3, SOURCEC4, SOURCEC5, SOURCEC6, SOURCEC7, SOURCEC8, SOURCEC9, SOURCED10, SOURCED11, SOURCED12, SOURCED13, SOURCED14, SOURCED15, SOURCED16, SOURCED17, SOURCED18, SOURCED19, SOURCED2, SOURCED20, SOURCED21, SOURCED22, SOURCED23, SOURCED24, SOURCED25, SOURCED3, SOURCED4, SOURCED5, SOURCED6, SOURCED7, SOURCED8, SOURCED9: TPWIRE, ellajameson-core:TP_TH_WIRE
- added JD10, JD11, JD12, JD13, JD14, JD15, JD16, JD17, JD18, JD19, JD2, JD20, JD21, JD22, JD23, JD24, JD25, JD3, JD4, JD5, JD6, JD7, JD8, JD9, JN10, JN11, JN12, JN13, JN14, JN15, JN16, JN17, JN18, JN19, JN2, JN20, JN21, JN22, JN23, JN24, JN25, JN3, JN4, JN5, JN6, JN7, JN8, JN9, JP10, JP11, JP12, JP13, JP14, JP15, JP16, JP17, JP18, JP19, JP2, JP20, JP21, JP22, JP23, JP24, JP25, JP3, JP4, JP5, JP6, JP7, JP8, JP9, JS10, JS11, JS12, JS13, JS14, JS15, JS16, JS17, JS18, JS19, JS2, JS20, JS21, JS22, JS23, JS24, JS25, JS3, JS4, JS5, JS6, JS7, JS8, JS9: SJ_NO, ellajameson-core:SJ_2S-NO
- added Q10, Q11, Q12, Q13, Q14, Q15, Q16, Q17, Q18, Q19, Q2, Q20, Q21, Q22, Q23, Q24, Q25, Q3, Q4, Q5, Q6, Q7, Q8, Q9: 2N7002, ellajameson-core:SOT23
- added R10, R11, R12, R13, R14, R15, R16, R17, R18, R19, R2, R20, R21, R22, R23, R24, R25, R3, R4, R5, R6, R7, R8, R9: (no value), ellajameson-core:R0603
Connections:
- new net GND: JN10.1, JN11.1, JN12.1, JN13.1, JN14.1, JN15.1, JN16.1, JN17.1, JN18.1, JN19.1, JN2.1, JN20.1, JN21.1, JN22.1, JN23.1, JN24.1, JN25.1, JN3.1, JN4.1, JN5.1, JN6.1, JN7.1, JN8.1, JN9.1
- new net N$1: D2.A, JP2.2, R2.1
- new net N$10: D3.C, DRAINA3.TP, DRAINB3.TP, DRAINC3.TP, DRAIND3.TP, JD3.2, JD4.1, JP3.1, JS12.1, Q3.3
- new net N$100: GATE25.TP, Q25.1
- new net N$11: JN3.2, JS3.2, Q3.2, SOURCEA3.TP, SOURCEB3.TP, SOURCEC3.TP, SOURCED3.TP
- new net N$12: GATE3.TP, Q3.1
- new net N$13: D4.A, JP4.2, R4.1
- new net N$14: D4.C, DRAINA4.TP, DRAINB4.TP, DRAINC4.TP, DRAIND4.TP, JD2.1, JD4.2, JP4.1, JS11.1, Q4.3
- new net N$15: JN4.2, JS4.2, Q4.2, SOURCEA4.TP, SOURCEB4.TP, SOURCEC4.TP, SOURCED4.TP
- new net N$16: GATE4.TP, Q4.1
- new net N$17: D5.A, JP5.2, R5.1
- new net N$18: D5.C, DRAINA5.TP, DRAINB5.TP, DRAINC5.TP, DRAIND5.TP, JD3.1, JD5.2, JP5.1, JS13.1, Q5.3
- new net N$19: JN5.2, JS5.2, Q5.2, SOURCEA5.TP, SOURCEB5.TP, SOURCEC5.TP, SOURCED5.TP
- new net N$2: D2.C, DRAINA2.TP, DRAINB2.TP, DRAINC2.TP, DRAIND2.TP, JD2.2, JP2.1, JS10.1, Q2.3
- new net N$20: GATE5.TP, Q5.1
- new net N$21: D6.A, JP6.2, R6.1
- new net N$22: D6.C, DRAINA6.TP, DRAINB6.TP, DRAINC6.TP, DRAIND6.TP, JD5.1, JD6.2, JP6.1, JS14.1, Q6.3
- new net N$23: JN6.2, JS6.2, Q6.2, SOURCEA6.TP, SOURCEB6.TP, SOURCEC6.TP, SOURCED6.TP
- new net N$24: GATE6.TP, Q6.1
- new net N$25: D7.A, JP7.2, R7.1
- new net N$26: D7.C, DRAINA7.TP, DRAINB7.TP, DRAINC7.TP, DRAIND7.TP, JD6.1, JD7.2, JP7.1, JS15.1, Q7.3
- new net N$27: JN7.2, JS7.2, Q7.2, SOURCEA7.TP, SOURCEB7.TP, SOURCEC7.TP, SOURCED7.TP
- new net N$28: GATE7.TP, Q7.1
- new net N$29: D8.A, JP8.2, R8.1
- new net N$3: JN2.2, JS2.2, Q2.2, SOURCEA2.TP, SOURCEB2.TP, SOURCEC2.TP, SOURCED2.TP
- new net N$30: D8.C, DRAINA8.TP, DRAINB8.TP, DRAINC8.TP, DRAIND8.TP, JD7.1, JD8.2, JP8.1, JS16.1, Q8.3
- new net N$31: JN8.2, JS8.2, Q8.2, SOURCEA8.TP, SOURCEB8.TP, SOURCEC8.TP, SOURCED8.TP
- new net N$32: GATE8.TP, Q8.1
- new net N$33: D9.A, JP9.2, R9.1
- new net N$34: D9.C, DRAINA9.TP, DRAINB9.TP, DRAINC9.TP, DRAIND9.TP, JD8.1, JD9.2, JP9.1, JS17.1, Q9.3
- new net N$35: JN9.2, JS9.2, Q9.2, SOURCEA9.TP, SOURCEB9.TP, SOURCEC9.TP, SOURCED9.TP
- new net N$36: GATE9.TP, Q9.1
- new net N$37: D10.A, JP10.2, R10.1
- new net N$38: D10.C, DRAINA10.TP, DRAINB10.TP, DRAINC10.TP, DRAIND10.TP, JD10.2, JP10.1, JS18.1, Q10.3
- new net N$39: JN10.2, JS10.2, Q10.2, SOURCEA10.TP, SOURCEB10.TP, SOURCEC10.TP, SOURCED10.TP
- new net N$4: GATE2.TP, Q2.1
- new net N$40: GATE10.TP, Q10.1
- new net N$41: D11.A, JP11.2, R11.1
- new net N$42: D11.C, DRAINA11.TP, DRAINB11.TP, DRAINC11.TP, DRAIND11.TP, JD10.1, JD11.2, JP11.1, JS19.1, Q11.3
- new net N$43: JN11.2, JS11.2, Q11.2, SOURCEA11.TP, SOURCEB11.TP, SOURCEC11.TP, SOURCED11.TP
- new net N$44: GATE11.TP, Q11.1
- new net N$45: D12.A, JP12.2, R12.1
- new net N$46: D12.C, DRAINA12.TP, DRAINB12.TP, DRAINC12.TP, DRAIND12.TP, JD11.1, JD12.2, JP12.1, JS20.1, Q12.3
- new net N$47: JN12.2, JS12.2, Q12.2, SOURCEA12.TP, SOURCEB12.TP, SOURCEC12.TP, SOURCED12.TP
- new net N$48: GATE12.TP, Q12.1
- new net N$49: D13.A, JP13.2, R13.1
- new net N$50: D13.C, DRAINA13.TP, DRAINB13.TP, DRAINC13.TP, DRAIND13.TP, JD12.1, JD13.2, JP13.1, JS21.1, Q13.3
- new net N$51: JN13.2, JS13.2, Q13.2, SOURCEA13.TP, SOURCEB13.TP, SOURCEC13.TP, SOURCED13.TP
- new net N$52: GATE13.TP, Q13.1
- new net N$53: D14.A, JP14.2, R14.1
- new net N$54: D14.C, DRAINA14.TP, DRAINB14.TP, DRAINC14.TP, DRAIND14.TP, JD13.1, JD14.2, JP14.1, JS22.1, Q14.3
- new net N$55: JN14.2, JS14.2, Q14.2, SOURCEA14.TP, SOURCEB14.TP, SOURCEC14.TP, SOURCED14.TP
- new net N$56: GATE14.TP, Q14.1
- new net N$57: D15.A, JP15.2, R15.1
- new net N$58: D15.C, DRAINA15.TP, DRAINB15.TP, DRAINC15.TP, DRAIND15.TP, JD14.1, JD15.2, JP15.1, JS23.1, Q15.3
- new net N$59: JN15.2, JS15.2, Q15.2, SOURCEA15.TP, SOURCEB15.TP, SOURCEC15.TP, SOURCED15.TP
- new net N$60: GATE15.TP, Q15.1
- new net N$61: D16.A, JP16.2, R16.1
- new net N$62: D16.C, DRAINA16.TP, DRAINB16.TP, DRAINC16.TP, DRAIND16.TP, JD15.1, JD16.2, JP16.1, JS24.1, Q16.3
- new net N$63: JN16.2, JS16.2, Q16.2, SOURCEA16.TP, SOURCEB16.TP, SOURCEC16.TP, SOURCED16.TP
- new net N$64: GATE16.TP, Q16.1
- new net N$65: D17.A, JP17.2, R17.1
- new net N$66: D17.C, DRAINA17.TP, DRAINB17.TP, DRAINC17.TP, DRAIND17.TP, JD16.1, JD17.2, JP17.1, JS25.1, Q17.3
- new net N$67: JN17.2, JS17.2, Q17.2, SOURCEA17.TP, SOURCEB17.TP, SOURCEC17.TP, SOURCED17.TP
- new net N$68: GATE17.TP, Q17.1
- new net N$69: D18.A, JP18.2, R18.1
- new net N$70: D18.C, DRAINA18.TP, DRAINB18.TP, DRAINC18.TP, DRAIND18.TP, JD18.2, JP18.1, Q18.3
- new net N$71: JN18.2, JS18.2, Q18.2, SOURCEA18.TP, SOURCEB18.TP, SOURCEC18.TP, SOURCED18.TP
- new net N$72: GATE18.TP, Q18.1
- new net N$73: D19.A, JP19.2, R19.1
- new net N$74: D19.C, DRAINA19.TP, DRAINB19.TP, DRAINC19.TP, DRAIND19.TP, JD18.1, JD19.2, JP19.1, Q19.3
- new net N$75: JN19.2, JS19.2, Q19.2, SOURCEA19.TP, SOURCEB19.TP, SOURCEC19.TP, SOURCED19.TP
- new net N$76: GATE19.TP, Q19.1
- new net N$77: D20.A, JP20.2, R20.1
- new net N$78: D20.C, DRAINA20.TP, DRAINB20.TP, DRAINC20.TP, DRAIND20.TP, JD19.1, JD20.2, JP20.1, Q20.3
- new net N$79: JN20.2, JS20.2, Q20.2, SOURCEA20.TP, SOURCEB20.TP, SOURCEC20.TP, SOURCED20.TP
- new net N$80: GATE20.TP, Q20.1
- new net N$81: D21.A, JP21.2, R21.1
- new net N$82: D21.C, DRAINA21.TP, DRAINB21.TP, DRAINC21.TP, DRAIND21.TP, JD20.1, JD21.2, JP21.1, Q21.3
- new net N$83: JN21.2, JS21.2, Q21.2, SOURCEA21.TP, SOURCEB21.TP, SOURCEC21.TP, SOURCED21.TP
- new net N$84: GATE21.TP, Q21.1
- new net N$85: D22.A, JP22.2, R22.1
- new net N$86: D22.C, DRAINA22.TP, DRAINB22.TP, DRAINC22.TP, DRAIND22.TP, JD21.1, JD22.2, JP22.1, Q22.3
- new net N$87: JN22.2, JS22.2, Q22.2, SOURCEA22.TP, SOURCEB22.TP, SOURCEC22.TP, SOURCED22.TP
- new net N$88: GATE22.TP, Q22.1
- new net N$89: D23.A, JP23.2, R23.1
- new net N$9: D3.A, JP3.2, R3.1
- new net N$90: D23.C, DRAINA23.TP, DRAINB23.TP, DRAINC23.TP, DRAIND23.TP, JD22.1, JD23.2, JP23.1, Q23.3
- new net N$91: JN23.2, JS23.2, Q23.2, SOURCEA23.TP, SOURCEB23.TP, SOURCEC23.TP, SOURCED23.TP
- new net N$92: GATE23.TP, Q23.1
- new net N$93: D24.A, JP24.2, R24.1
- new net N$94: D24.C, DRAINA24.TP, DRAINB24.TP, DRAINC24.TP, DRAIND24.TP, JD23.1, JD24.2, JP24.1, Q24.3
- new net N$95: JN24.2, JS24.2, Q24.2, SOURCEA24.TP, SOURCEB24.TP, SOURCEC24.TP, SOURCED24.TP
- new net N$96: GATE24.TP, Q24.1
- new net N$97: D25.A, JP25.2, R25.1
- new net N$98: D25.C, DRAINA25.TP, DRAINB25.TP, DRAINC25.TP, DRAIND25.TP, JD24.1, JD25.2, JP25.1, Q25.3
- new net N$99: JN25.2, JS25.2, Q25.2, SOURCEA25.TP, SOURCEB25.TP, SOURCEC25.TP, SOURCED25.TP
- new net VCC: R10.2, R11.2, R12.2, R13.2, R14.2, R15.2, R16.2, R17.2, R18.2, R19.2, R2.2, R20.2, R21.2, R22.2, R23.2, R24.2, R25.2, R3.2, R4.2, R5.2, R6.2, R7.2, R8.2, R9.2
Routing:
- net VCC: track 0.00 -> 227.5 mm, vias 0 -> 24
- net GND: track 0.00 -> 73.6 mm, vias 0 -> 24
- net N$42: track 0.00 -> 16.2 mm
- net N$54: track 0.00 -> 16.0 mm
- net N$66: track 0.00 -> 15.8 mm
- net N$34: track 0.00 -> 15.8 mm
- net N$58: track 0.00 -> 15.8 mm
- net N$30: track 0.00 -> 15.8 mm
- net N$26: track 0.00 -> 15.8 mm
- net N$62: track 0.00 -> 15.8 mm
- net N$46: track 0.00 -> 15.8 mm
- net N$14: track 0.00 -> 15.8 mm
- net N$10: track 0.00 -> 15.8 mm
- net N$22: track 0.00 -> 15.8 mm
- net N$18: track 0.00 -> 15.8 mm
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- added copper zone on layer 16, net GND
Other:
- board outline added: 49.5 x 66 mm
- board text added: "#X"
- board text added: "D"
- board text added: "G"
- board text added: "S"
