File: Eagle/PCBs/NMOS Experimenter Board/experimenter.brd (EAGLE design)
At the start: 77.5 x 99.1 mm, 1182 parts, among them Q10 2N7002, Q11 2N7002, Q12 2N7002, Q13 2N7002, Q14 2N7002, Q15 2N7002, Q16 2N7002, Q17 2N7002, Q18 2N7002, Q19 2N7002, Q2 2N7002, Q20 2N7002, Q21 2N7002, Q22 2N7002, Q23 2N7002, Q24 2N7002, Q25 2N7002, Q26 2N7002, Q27 2N7002, Q28 2N7002, Q29 2N7002, Q3 2N7002, Q30 2N7002, Q31 2N7002, Q32 2N7002, Q33 2N7002, Q34 2N7002, Q35 2N7002, Q36 2N7002, Q37 2N7002, Q38 2N7002, Q39 2N7002, Q4 2N7002, Q40 2N7002, Q41 2N7002, Q42 2N7002, Q43 2N7002, Q44 2N7002, Q45 2N7002, Q46 2N7002, Q47 2N7002, Q48 2N7002, Q49 2N7002, Q5 2N7002, Q50 2N7002, Q51 2N7002, Q52 2N7002, Q53 2N7002, Q54 2N7002, Q55 2N7002, Q56 2N7002, Q57 2N7002, Q58 2N7002, Q59 2N7002, Q6 2N7002, Q60 2N7002, Q61 2N7002, Q62 2N7002, Q63 2N7002, Q64 2N7002, Q65 2N7002, Q66 2N7002, Q67 2N7002, Q68 2N7002, Q69 2N7002, Q7 2N7002, Q70 2N7002, Q71 2N7002, Q72 2N7002, Q73 2N7002, Q8 2N7002, Q9 2N7002, U1 74HC14PW

Commit message: Update experimenter.brd
Parts:
- turned J1 to 270 degrees
Routing:
- net VCC: track 764.0 -> 769.5 mm
Changed lines of the file:
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@@
 </layers>
 <board>
-<fusionsync huburn="a.cGVyc29uYWw6dWUyZGY0M2Ex" projecturn="a.cGVyc29uYWw6dWUyZGY0M2ExIzIwMjMwNDIzNjMzMDQzOTMx" f3durn="urn:adsk.wipprod:dm.lineage:ybcwFhw2S7Sfdtd4-gzlww" pcbguid="" lastpulledtime="" lastsyncedchangeguid="" latestrevisionid="611b4f10-5022-4631-9896-331b126fc531" lastsyncedrevisionid="611b4f10-5022-4631-9896-331b126fc531" lastboardhashguid="81255f3b-b9e8-1c72-a19b-cfd540b0dd78" lastpushedtime="2023-04-23T11:59:13Z" linktopcb3d="true"/>
+<fusionsync huburn="a.cGVyc29uYWw6dWUyZGY0M2Ex" projecturn="a.cGVyc29uYWw6dWUyZGY0M2ExIzIwMjMwNDIzNjMzMDQzOTMx" f3durn="urn:adsk.wipprod:dm.lineage:ybcwFhw2S7Sfdtd4-gzlww" pcbguid="" lastpulledtime="" lastsyncedchangeguid="" latestrevisionid="d7e2e287-3d4f-4587-b865-e3116f039d92" lastsyncedrevisionid="d7e2e287-3d4f-4587-b865-e3116f039d92" lastboardhashguid="c5c264f8-329d-c11c-44e9-3ba24df78021" lastpushedtime="2023-04-23T13:07:44Z" linktopcb3d="true"/>
 <plain>
 <wire x1="0" y1="0" x2="0" y2="99.06" width="0.0762" layer="20"/>
@@
 <element name="B5" library="ellajameson-core" library_urn="urn:adsk.eagle:library:3740209" package="TP_TH_WIRE" package3d_urn="urn:adsk.eagle:package:40139460/2" value="TPWIRE" x="31.75" y="87.63" smashed="yes"/>
 <element name="B6" library="ellajameson-core" library_urn="urn:adsk.eagle:library:3740209" package="TP_TH_WIRE" package3d_urn="urn:adsk.eagle:package:40139460/2" value="TPWIRE" x="36.83" y="87.63" smashed="yes"/>
-<element name="J1" library="ellajameson-core" library_urn="urn:adsk.eagle:library:3740209" package="OSTVN02A150" package3d_urn="urn:adsk.eagle:package:12594929/2" value="" x="73.66" y="41.91" smashed="yes" rot="R90"/>
+<element name="J1" library="ellajameson-core" library_urn="urn:adsk.eagle:library:3740209" package="OSTVN02A150" package3d_urn="urn:adsk.eagle:package:12594929/2" value="" x="73.66" y="41.91" smashed="yes" rot="R270"/>
 <element name="C1" library="ellajameson-core" library_urn="urn:adsk.eagle:library:3740209" package="C0603" package3d_urn="urn:adsk.eagle:package:7587834/2" value="0.1u" x="14.986" y="83.439" smashed="yes" rot="R180"/>
 <element name="C4" library="ellajameson-core" library_urn="urn:adsk.eagle:library:3740209" package="C0603" package3d_urn="urn:adsk.eagle:package:7587834/2" value="0.1u" x="74.93" y="45.72" smashed="yes" rot="R180"/>
@@
 <wire x1="64.389" y1="42.164" x2="67.23846875" y2="42.164" width="0.3048" layer="16"/>
 <wire x1="67.23846875" y1="42.164" x2="67.58926875" y2="42.5148" width="0.3048" layer="16"/>
-<wire x1="71.12" y1="43.18" x2="73.66" y2="43.18" width="0.3048" layer="16"/>
-<wire x1="71.12" y1="43.18" x2="70.4548" y2="42.5148" width="0.3048" layer="16"/>
-<wire x1="67.58926875" y1="42.5148" x2="70.4548" y2="42.5148" width="0.3048" layer="16"/>
-<wire x1="73.66" y1="43.18" x2="74.08" y2="43.6" width="0.3048" layer="1"/>
-<wire x1="74.08" y1="43.6" x2="74.08" y2="45.72" width="0.3048" layer="1"/>
 <contactref element="SJ2" pad="1"/>
 <wire x1="74.08" y1="45.72" x2="73.152" y2="45.72" width="0.3048" layer="1"/>
 <wire x1="72.39" y1="46.482" x2="72.39" y2="47.752" width="0.3048" layer="1"/>
 <wire x1="73.152" y1="45.72" x2="72.39" y2="46.482" width="0.3048" layer="1"/>
+<wire x1="67.58926875" y1="42.5148" x2="69.57073125" y2="42.5148" width="0.3048" layer="16"/>
+<wire x1="71.44553125" y1="40.64" x2="73.66" y2="40.64" width="0.3048" layer="16"/>
+<wire x1="69.57073125" y1="42.5148" x2="71.44553125" y2="40.64" width="0.3048" layer="16"/>
+<wire x1="73.66" y1="40.64" x2="72.39" y2="40.64" width="0.3048" layer="1"/>
+<wire x1="72.39" y1="40.64" x2="71.12" y2="41.91" width="0.3048" layer="1"/>
+<wire x1="71.12" y1="41.91" x2="71.12" y2="43.688" width="0.3048" layer="1"/>
+<wire x1="71.12" y1="43.688" x2="73.152" y2="45.72" width="0.3048" layer="1"/>
 </signal>
 <signal name="N$69">

Commit message: Added switches, preemptive first version
Parts:
- added C10, C12, C13, C14, C15, C6, C8: 0.1u, ellajameson-core:C0603
- added R1, R74, R79, R80, R83, R84, R87, R88, R91, R92, R95, R96: 10k, ellajameson-core:R0603
- added SO1, SO2, SO3, SO4, SO5, SO6: TPWIRE, ellajameson-core:TP_TH_WIRE
- added SW1: (no value), ellajameson-core:EDG-06
- added U2: 74HC14PW, ellajameson-core:TSSOP14
Connections:
- new net N$307: SO6.TP, U2.12
- new net N$308: SO5.TP, U2.10
- new net N$311: SO4.TP, U2.8
- new net N$312: C8.1, R80.1, U2.3
- new net N$313: SO3.TP, U2.6
- new net N$314: C10.1, R84.1, U2.5
- new net N$315: SO2.TP, U2.4
- new net N$316: C12.1, R88.1, U2.9
- new net N$317: SO1.TP, U2.2
- new net N$318: C13.1, R92.1, U2.11
- new net N$320: C14.1, R96.1, U2.13
- new net S1F: C6.1, R74.1, U2.1
- new net S1G: R1.1, R74.2, SW1.12
- new net S2G: R79.1, R80.2, SW1.11
- new net S3G: R83.1, R84.2, SW1.10
- new net S4G: R87.1, R88.2, SW1.9
- new net S5G: R91.1, R92.2, SW1.8
- new net S6G: R95.1, R96.2, SW1.7
- net GND: now also C10.2, C12.2, C13.2, C14.2, C15.2, C6.2, C8.2, SW1.1, SW1.2, SW1.3, SW1.4, SW1.5, SW1.6, U2.7
- net VCC: now also C15.1, R1.2, R79.2, R83.2, R87.2, R91.2, R95.2, U2.14
Routing:
- net VCC: track 769.5 -> 827.2 mm, vias 78 -> 84
- net S6G: track 0.00 -> 37.9 mm, vias 0 -> 2
- net N$307: track 0.00 -> 34.9 mm, vias 0 -> 1
- net N$308: track 0.00 -> 30.8 mm, vias 0 -> 1
- net N$313: track 0.00 -> 27.6 mm, vias 0 -> 1
- net N$315: track 0.00 -> 26.8 mm, vias 0 -> 1
- net N$311: track 0.00 -> 25.6 mm, vias 0 -> 1
- net N$317: track 0.00 -> 24.2 mm, vias 0 -> 1
- net S1F: track 0.00 -> 22.1 mm
- net S5G: track 0.00 -> 19.2 mm
- net GND: track 268.9 -> 287.6 mm, vias 87 -> 96
- net N$312: track 0.00 -> 17.8 mm
- net S4G: track 0.00 -> 15.4 mm
- net N$314: track 0.00 -> 14.4 mm
- net N$318: track 0.00 -> 13.8 mm, vias 0 -> 2
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Other:
- board text added: "+5V"
- board text added: "NMOS Laboratory Board v1 by Ella Jameson"
- board text added: "SW1"
- board text added: "SW2"
- board text added: "SW3"
- board text added: "SW4"
- board text added: "SW5"
- board text added: "SW6"
